Commit message: Push local changes

File: resources/robots/rhea/urdf/rhea.urdf (robot description, URDF)
Before this commit: robot rhea, 8 links, 7 joints
Links:
- removed link imu
- removed link left_hip
- removed link left_knee
- removed link right_hip
- removed link right_knee
- added link left_leg, mass 0.1
- added link right_leg, mass 0.1
Joints:
- removed joint imu
- removed joint left_hip
- removed joint left_knee
- removed joint right_hip
- removed joint right_knee
- added joint left_leg: type prismatic, parent base_link, child left_leg, origin xyz=0 0.1 0 rpy=0 0 3.1415, axis 0 0 1.0, limit lower=-0.35 upper=-0.075 effort=100.0 velocity=1.0
- added joint right_leg: type prismatic, parent base_link, child right_leg, origin xyz=0 -0.1 0 rpy=0 0 0, axis 0 0 1.0, limit lower=-0.35 upper=-0.075 effort=100.0 velocity=1.0
- joint left_wheel: limit effort=9.0 velocity=42.0 -> lower=-100000 upper=100000 effort=9.0 velocity=42.0; origin xyz=0.225 0 0 rpy=0 0 0 -> xyz=0 0 0 rpy=1.5708 1.5708 0; parent left_knee -> left_leg; type continuous -> revolute
- joint right_wheel: limit effort=9.0 velocity=42.0 -> lower=-100000 upper=100000 effort=9.0 velocity=42.0; origin xyz=0.225 0 0 rpy=0 0 0 -> xyz=0 0 0 rpy=1.5708 1.5708 0; parent right_knee -> right_leg; type continuous -> revolute

Commit message: Fix more issues in the URDF

File: resources/robots/rhea/urdf/rhea.urdf (robot description, URDF)
Before this commit: robot rhea, 5 links, 4 joints
Links:
- link base_link: mass 3.0 -> 5.0

Commit message: Push changes

File: resources/robots/rhea/urdf/rhea.urdf (robot description, URDF)
Before this commit: robot rhea, 5 links, 4 joints
Links:
- removed link left_leg
- removed link right_leg
- added link imu, mass 0.001
- added link left_hip, mass 1.0; collision box size=0.05693 0.0756 0.30004
- added link left_knee, mass 0.5; collision box size=0.05693 0.028 0.30004
- added link right_hip, mass 1.0; collision box size=0.05693 0.0756 0.30004
- added link right_knee, mass 0.5; collision box size=0.05693 0.028 0.30004
- link base_link: mass 5.0 -> 4.0; geometry collision box size=0.216 0.14 0.231
- link left_wheel: mass 0.4 -> 1.0; geometry collision cylinder length=0.048 radius=0.11
- link right_wheel: mass 0.4 -> 1.0; geometry collision cylinder length=0.048 radius=0.11
Joints:
- removed joint left_leg
- removed joint right_leg
- added joint imu: type fixed, parent base_link, child imu, origin xyz=0 0 0 rpy=1.5708 0 -1.5708
- added joint left_hip: type revolute, parent base_link, child left_hip, origin xyz=0 0.1255 0 rpy=-1.5708 1.5708 0, axis 0 0 1.0, limit lower=-0.68068 upper=2.46091 effort=35.0 velocity=26.0
- added joint left_knee: type revolute, parent left_hip, child left_knee, origin xyz=0.25 0 0 rpy=0 0 0, axis 0 0 1.0, limit lower=-2.75762 upper=-0.66323 effort=35.0 velocity=26.0
- added joint right_hip: type revolute, parent base_link, child right_hip, origin xyz=0 -0.1255 0 rpy=1.5708 1.5708 0, axis 0 0 1.0, limit lower=-2.46091 upper=0.68068 effort=35.0 velocity=26.0
- added joint right_knee: type revolute, parent right_hip, child right_knee, origin xyz=0.25 0 0 rpy=0 0 0, axis 0 0 1.0, limit lower=0.66323 upper=2.75762 effort=35.0 velocity=26.0
- joint left_wheel: limit lower=-100000 upper=100000 effort=9.0 velocity=42.0 -> lower=-100000.0 upper=100000.0 effort=2.0 velocity=250.0; origin xyz=0 0 0 rpy=1.5708 1.5708 0 -> xyz=0.25 0 0 rpy=0 0 0; parent left_leg -> left_knee
- joint right_wheel: limit lower=-100000 upper=100000 effort=9.0 velocity=42.0 -> lower=-100000.0 upper=100000.0 effort=2.0 velocity=250.0; origin xyz=0 0 0 rpy=1.5708 1.5708 0 -> xyz=0.25 0 0 rpy=0 0 0; parent right_leg -> right_knee
