Commit message: Update Pupper v3 URDF

File: resources/robots/pupper/urdf/pupper_v3.urdf (robot description, URDF)
Before this commit: robot pupper_v3, 13 links, 12 joints
Links:
- link base_link: mass 1.2 -> 1.0
- link leg_back_l_1: mass 0.16 -> 0.2; geometry collision cylinder length=0.025 radius=0.0265; visual mesh filename=../meshes/dae/pupperv3_export.011.dae scale=1.0 1.0 1.0
- link leg_back_l_2: mass 0.02 -> 0.2; geometry collision box size=0.07978 0.03123 0.02896; collision cylinder length=0.025 radius=0.0265
- link leg_back_l_3: geometry collision box size=0.06966 0.01583 0.01448; collision sphere radius=0.01984
- link leg_back_r_1: mass 0.16 -> 0.2; geometry collision cylinder length=0.025 radius=0.0265; visual mesh filename=../meshes/dae/pupperv3_export.010.dae scale=1.0 1.0 1.0
- link leg_back_r_2: mass 0.02 -> 0.2; geometry collision box size=0.07978 0.03123 0.02896; collision cylinder length=0.025 radius=0.0265
- link leg_back_r_3: geometry collision box size=0.06966 0.01583 0.01448; collision sphere radius=0.01984
- link leg_front_l_1: mass 0.16 -> 0.2; geometry collision cylinder length=0.025 radius=0.0265; visual mesh filename=../meshes/dae/pupperv3_export.012.dae scale=1.0 1.0 1.0
- link leg_front_l_2: mass 0.17 -> 0.2; geometry collision box size=0.07978 0.03123 0.02896; collision cylinder length=0.025 radius=0.0265
- link leg_front_l_3: geometry collision box size=0.06966 0.01583 0.01448; collision sphere radius=0.01984
- link leg_front_r_1: mass 0.16 -> 0.2; geometry collision cylinder length=0.025 radius=0.0265; visual mesh filename=../meshes/dae/pupperv3_export.009.dae scale=1.0 1.0 1.0
- link leg_front_r_2: mass 0.02 -> 0.2; geometry collision box size=0.07978 0.03123 0.02896; collision cylinder length=0.025 radius=0.0265
- link leg_front_r_3: geometry collision box size=0.06966 0.01583 0.01448; collision sphere radius=0.01984
Joints:
- joint leg_back_l_1: limit lower=-2.87979 upper=2.35619 effort=3.7 velocity=47.12389 -> lower=-2.0944 upper=1.22173 effort=3.7 velocity=47.12389
- joint leg_back_l_2: limit lower=-1.5708 upper=0.69813 effort=3.7 velocity=47.12389 -> lower=-0.87266 upper=0.5236 effort=3.7 velocity=47.12389
- joint leg_back_l_3: limit lower=-1.20428 upper=3.14159 effort=3.7 velocity=47.12389 -> lower=-0.82903 upper=3.05433 effort=3.7 velocity=47.12389
- joint leg_back_r_1: limit lower=-2.35619 upper=2.87979 effort=3.7 velocity=47.12389 -> lower=-1.22173 upper=2.0944 effort=3.7 velocity=47.12389
- joint leg_back_r_2: limit lower=-0.69813 upper=1.5708 effort=3.7 velocity=47.12389 -> lower=-0.5236 upper=0.87266 effort=3.7 velocity=47.12389
- joint leg_back_r_3: limit lower=-3.14159 upper=1.20428 effort=3.7 velocity=47.12389 -> lower=-3.05433 upper=0.82903 effort=3.7 velocity=47.12389
- joint leg_front_l_1: limit lower=-2.87979 upper=2.35619 effort=3.7 velocity=47.12389 -> lower=-2.0944 upper=1.22173 effort=3.7 velocity=47.12389
- joint leg_front_l_2: limit lower=-1.5708 upper=0.69813 effort=3.7 velocity=47.12389 -> lower=-0.87266 upper=0.5236 effort=3.7 velocity=47.12389
- joint leg_front_l_3: limit lower=-1.20428 upper=3.14159 effort=3.7 velocity=47.12389 -> lower=-0.82903 upper=3.05433 effort=3.7 velocity=47.12389
- joint leg_front_r_1: limit lower=-2.35619 upper=2.87979 effort=3.7 velocity=47.12389 -> lower=-1.22173 upper=2.0944 effort=3.7 velocity=47.12389
- joint leg_front_r_2: limit lower=-0.69813 upper=1.5708 effort=3.7 velocity=47.12389 -> lower=-0.5236 upper=0.87266 effort=3.7 velocity=47.12389
- joint leg_front_r_3: limit lower=-3.14159 upper=1.20428 effort=3.7 velocity=47.12389 -> lower=-3.05433 upper=0.82903 effort=3.7 velocity=47.12389

Commit message: fix collision and weird inertia

File: resources/robots/pupper/urdf/pupper_v3.urdf (robot description, URDF)
Before this commit: robot pupper_v3, 13 links, 12 joints
Links:
- link base_link: geometry collision box size=0.26419 0.13252 0.11; visual mesh filename=../meshes/dae/pupperv3_export.dae scale=1.0 1.0 1.0
